Commit message: Rename omniquad12 leg joint names

File: src/pi3hat/pi3hat_hw_interface/urdf/omniquad12.xacro (robot description, xacro)
@@ -1,5 +1,5 @@
 <?xml version="1.0" ?>
 <robot name="omnicar"  xmlns:xacro="http://ros.org/wiki/xacro">
-    <xacro:macro name="wheel_joint" params="name id bus second_encoder_source max_pos_limit min_pos_limit actuator_trasmission">
+    <xacro:macro name="joint" params="name id bus second_encoder_source max_pos_limit min_pos_limit actuator_trasmission">
         <joint name="${name}">
             <param name="id">${id}</param>
@@ -39,4 +39,10 @@
         </joint>
     </xacro:macro>
+    <xacro:macro name="leg_joint" params="name id bus">
+        <xacro:joint name="${name}" id="${id}" bus="${bus}" second_encoder_source="-1" max_pos_limit="3.14" min_pos_limit="-3.14" actuator_trasmission="9"/>
+    </xacro:macro>
+    <xacro:macro name="wheel_joint" params="name id bus">
+        <xacro:joint name="${name}" id="${id}" bus="${bus}" second_encoder_source="-1" max_pos_limit="5000.0" min_pos_limit="-5000.0" actuator_trasmission="15"/>
+    </xacro:macro>
     <xacro:macro name="distributor_joint" params="name id">
         <joint name="${name}">
@@ -68,16 +74,16 @@
             <param name="attitude_hz">400</param>
         </hardware>
-        <xacro:wheel_joint name="LF_HIP_JNT" id="1" bus="3" second_encoder_source = "-1" max_pos_limit ="3.14" min_pos_limit ="-3.14" actuator_trasmission = "9"/>
-        <xacro:wheel_joint name="LF_KNEE_JNT" id="2" bus="3" second_encoder_source = "-1" max_pos_limit ="3.14" min_pos_limit ="-3.14" actuator_trasmission = "9"/>
-        <xacro:wheel_joint name="RF_HIP_JNT" id="3" bus="4" second_encoder_source = "-1" max_pos_limit ="3.14" min_pos_limit ="-3.14" actuator_trasmission = "9"/>
-        <xacro:wheel_joint name="RF_KNEE_JNT" id="4" bus="4" second_encoder_source = "-1" max_pos_limit ="3.14" min_pos_limit ="-3.14" actuator_trasmission = "9"/>
-        <xacro:wheel_joint name="LH_HIP_JNT" id="5" bus="1" second_encoder_source = "-1" max_pos_limit ="3.14" min_pos_limit ="-3.14" actuator_trasmission = "9"/>
-        <xacro:wheel_joint name="LH_KNEE_JNT" id="6" bus="1" second_encoder_source = "-1" max_pos_limit ="3.14" min_pos_limit ="-3.14" actuator_trasmission = "9"/>
-        <xacro:wheel_joint name="RH_HIP_JNT" id="7" bus="2" second_encoder_source = "-1" max_pos_limit ="3.14" min_pos_limit ="-3.14" actuator_trasmission = "9"/>
-        <xacro:wheel_joint name="RH_KNEE_JNT" id="8" bus="2" second_encoder_source = "-1" max_pos_limit ="3.14" min_pos_limit ="-3.14" actuator_trasmission = "9"/>
-        <xacro:wheel_joint name="LF_WHEEL_JNT" id="9" bus="3" second_encoder_source = "-1" max_pos_limit ="5000.0" min_pos_limit ="-5000.0" actuator_trasmission = "15"/>
-        <xacro:wheel_joint name="RF_WHEEL_JNT" id="10" bus="4" second_encoder_source = "-1" max_pos_limit ="5000.0" min_pos_limit ="-5000.0" actuator_trasmission = "15"/>
-        <xacro:wheel_joint name="RH_WHEEL_JNT" id="12" bus="2" second_encoder_source = "-1" max_pos_limit ="5000.0" min_pos_limit ="-5000.0" actuator_trasmission = "15"/>
-        <xacro:wheel_joint name="LH_WHEEL_JNT" id="11" bus="1" second_encoder_source = "-1" max_pos_limit ="5000.0" min_pos_limit ="-5000.0" actuator_trasmission = "15"/>
+        <xacro:leg_joint name="LF_HFE" id="1" bus="3"/>
+        <xacro:leg_joint name="LF_KFE" id="2" bus="3"/>
+        <xacro:leg_joint name="RF_HFE" id="3" bus="4"/>
+        <xacro:leg_joint name="RF_KFE" id="4" bus="4"/>
+        <xacro:leg_joint name="LH_HFE" id="5" bus="1"/>
+        <xacro:leg_joint name="LH_KFE" id="6" bus="1"/>
+        <xacro:leg_joint name="RH_HFE" id="7" bus="2"/>
+        <xacro:leg_joint name="RH_KFE" id="8" bus="2"/>
+        <xacro:wheel_joint name="LF_WHEEL_JNT" id="9" bus="3"/>
+        <xacro:wheel_joint name="RF_WHEEL_JNT" id="10" bus="4"/>
+        <xacro:wheel_joint name="RH_WHEEL_JNT" id="12" bus="2"/>
+        <xacro:wheel_joint name="LH_WHEEL_JNT" id="11" bus="1"/>
         <xacro:distributor_joint name="Distributor_L" id="32"/>
         <xacro:distributor_joint name="Distributor_R" id="33"/>
