Commit message: Update config files

File: src/pi3hat/pi3hat_hw_interface/urdf/omnicar.xacro (robot description, xacro)
@@ -28,7 +28,7 @@
             <param name="d_current_res">0</param>
             <param name="abs_position_res">0</param>
-            <param name="power_res">0</param>
+            <param name="power_res">8</param>
             <param name="motor_temperature_res">0</param>
-            <param name="voltage_res">0</param>
+            <param name="voltage_res">16</param>
             <param name="temperature_res">8</param>
             <param name="position_error_res">64</param>
@@ -68,8 +68,8 @@
             <param name="attitude_hz">400</param>
         </hardware>
-        <xacro:wheel_joint name="LF_WHEEL_JNT" id="3" bus="2"/>
-        <xacro:wheel_joint name="RF_WHEEL_JNT" id="5" bus="4"/>
-        <xacro:wheel_joint name="RH_WHEEL_JNT" id="7" bus="3"/>
-        <xacro:wheel_joint name="LH_WHEEL_JNT" id="9" bus="1"/>
+        <xacro:wheel_joint name="LF_WHEEL" id="3" bus="2"/>
+        <xacro:wheel_joint name="RF_WHEEL" id="5" bus="4"/>
+        <xacro:wheel_joint name="LH_WHEEL" id="9" bus="1"/>
+        <xacro:wheel_joint name="RH_WHEEL" id="7" bus="3"/>
         <xacro:distributor_joint name="Distributor_L" id="32"/>
         <xacro:distributor_joint name="Distributor_R" id="33"/>

File: src/pi3hat/pi3hat_hw_interface/urdf/omniquad12.xacro (robot description, xacro)
@@ -1,5 +1,5 @@
 <?xml version="1.0" ?>
 <robot name="omnicar"  xmlns:xacro="http://ros.org/wiki/xacro">
-    <xacro:macro name="joint" params="name id bus second_encoder_source max_pos_limit min_pos_limit actuator_trasmission">
+    <xacro:macro name="joint" params="name id bus kp kd second_encoder_source max_pos_limit min_pos_limit actuator_trasmission">
         <joint name="${name}">
             <param name="id">${id}</param>
@@ -7,6 +7,6 @@
             <param name="second_encoder_source">${second_encoder_source}</param>
             <param name="type">motor</param>
-            <param name="KP">5.0</param>
-            <param name="KD">0.1</param>
+            <param name="KP">${kp}</param>
+            <param name="KD">${kd}</param>
             <param name="KI">0.0</param>
             <param name="ilimit">0.0</param>
@@ -28,7 +28,7 @@
             <param name="d_current_res">0</param>
             <param name="abs_position_res">0</param>
-            <param name="power_res">0</param>
+            <param name="power_res">8</param>
             <param name="motor_temperature_res">0</param>
-            <param name="voltage_res">0</param>
+            <param name="voltage_res">16</param>
             <param name="temperature_res">8</param>
             <param name="position_error_res">64</param>
@@ -40,8 +40,8 @@
     </xacro:macro>
     <xacro:macro name="leg_joint" params="name id bus">
-        <xacro:joint name="${name}" id="${id}" bus="${bus}" second_encoder_source="-1" max_pos_limit="3.14" min_pos_limit="-3.14" actuator_trasmission="9"/>
+        <xacro:joint name="${name}" id="${id}" bus="${bus}" kp="100.0" kd="1.0" second_encoder_source="-1" max_pos_limit="3.14" min_pos_limit="-3.14" actuator_trasmission="9"/>
     </xacro:macro>
     <xacro:macro name="wheel_joint" params="name id bus">
-        <xacro:joint name="${name}" id="${id}" bus="${bus}" second_encoder_source="-1" max_pos_limit="5000.0" min_pos_limit="-5000.0" actuator_trasmission="15"/>
+        <xacro:joint name="${name}" id="${id}" bus="${bus}" kp="0.0" kd="1.0" second_encoder_source="-1" max_pos_limit="5000.0" min_pos_limit="-5000.0" actuator_trasmission="15"/>
     </xacro:macro>
     <xacro:macro name="distributor_joint" params="name id">
@@ -74,16 +74,16 @@
             <param name="attitude_hz">400</param>
         </hardware>
-        <xacro:leg_joint name="LF_HFE" id="1" bus="3"/>
-        <xacro:leg_joint name="LF_KFE" id="2" bus="3"/>
-        <xacro:leg_joint name="RF_HFE" id="3" bus="4"/>
-        <xacro:leg_joint name="RF_KFE" id="4" bus="4"/>
-        <xacro:leg_joint name="LH_HFE" id="5" bus="1"/>
-        <xacro:leg_joint name="LH_KFE" id="6" bus="1"/>
-        <xacro:leg_joint name="RH_HFE" id="7" bus="2"/>
-        <xacro:leg_joint name="RH_KFE" id="8" bus="2"/>
-        <xacro:wheel_joint name="LF_WHEEL_JNT" id="9" bus="3"/>
-        <xacro:wheel_joint name="RF_WHEEL_JNT" id="10" bus="4"/>
-        <xacro:wheel_joint name="RH_WHEEL_JNT" id="12" bus="2"/>
-        <xacro:wheel_joint name="LH_WHEEL_JNT" id="11" bus="1"/>
+        <xacro:leg_joint name="LF_HFE" id="3" bus="2"/>
+        <xacro:leg_joint name="LF_KFE" id="4" bus="2"/>
+        <xacro:leg_joint name="RF_HFE" id="5" bus="4"/>
+        <xacro:leg_joint name="RF_KFE" id="6" bus="4"/>
+        <xacro:leg_joint name="LH_HFE" id="9" bus="1"/>
+        <xacro:leg_joint name="LH_KFE" id="10" bus="1"/>
+        <xacro:leg_joint name="RH_HFE" id="7" bus="3"/>
+        <xacro:leg_joint name="RH_KFE" id="8" bus="3"/>
+        <xacro:wheel_joint name="LF_WHEEL" id="11" bus="2"/>
+        <xacro:wheel_joint name="RF_WHEEL" id="12" bus="4"/>
+        <xacro:wheel_joint name="LH_WHEEL" id="14" bus="1"/>
+        <xacro:wheel_joint name="RH_WHEEL" id="13" bus="3"/>
         <xacro:distributor_joint name="Distributor_L" id="32"/>
         <xacro:distributor_joint name="Distributor_R" id="33"/>
