Commit message: Fix interface's problems  to set params from xacro

File: src/pi3hat/pi3hat_hw_interface/urdf/SoftLeg.xacro (robot description, xacro)
@@ -1,5 +1,5 @@
 <?xml version="1.0" ?>
 <robot name="softleg" xmlns:xacro="http://ros.org/wiki/xacro">
-    <xacro:macro name="joint" params="name id bus kp kd second_encoder_source max_pos_limit min_pos_limit actuator_trasmission position_offset">
+    <xacro:macro name="joint" params="name id bus kp kd second_encoder_source max_pos_limit min_pos_limit actuator_trasmission position_offset max_current_A">
         <joint name="${name}">
             <param name="id">${id}</param>
@@ -23,5 +23,5 @@
             <param name="second_encoder_trasmission">3.23076923</param>
             <param name="max_power_W">450</param>
-            <param name="max_current_A">40</param>
+            <param name="max_current_A">${max_current_A}</param>
             <param name="position_res">64</param>
             <param name="velocity_res">64</param>
@@ -47,5 +47,5 @@
                      max_pos_limit="3.14" min_pos_limit="-3.14"
                      actuator_trasmission="9"
-                     position_offset="${position_offset}"/>
+                     position_offset="${position_offset}" max_current_A="80.0"/>
     </xacro:macro>
     <xacro:macro name="distributor_joint" params="name id">

File: src/pi3hat/pi3hat_hw_interface/urdf/arm.xacro (robot description, xacro)
@@ -1,5 +1,5 @@
 <?xml version="1.0" ?>
 <robot name="omnicar"  xmlns:xacro="http://ros.org/wiki/xacro">
-    <xacro:macro name="joint" params="name id bus kp kd second_encoder_source max_pos_limit min_pos_limit actuator_trasmission">
+    <xacro:macro name="joint" params="name id bus kp kd second_encoder_source max_pos_limit min_pos_limit actuator_trasmission max_current_A">
         <joint name="${name}">
             <param name="id">${id}</param>
@@ -23,5 +23,5 @@
             <param name="second_encoder_trasmission">3.23076923</param>
             <param name="max_power_W">450</param>
-            <param name="max_current_A">40</param>
+            <param name="max_current_A">${max_current_A}</param>
             <param name="position_res">64</param>
             <param name="velocity_res">64</param>
@@ -42,8 +42,8 @@
     </xacro:macro>
     <xacro:macro name="arm_joint" params="name id bus">
-        <xacro:joint name="${name}" id="${id}" bus="${bus}" kp="100.0" kd="1.0" second_encoder_source="-1" max_pos_limit="3.14" min_pos_limit="-3.14" actuator_trasmission="9"/>
+        <xacro:joint name="${name}" id="${id}" bus="${bus}" kp="100.0" kd="1.0" second_encoder_source="-1" max_pos_limit="3.14" min_pos_limit="-3.14" actuator_trasmission="9" max_current_A="80.0"/>
     </xacro:macro>
     <xacro:macro name="wheel_joint" params="name id bus">
-        <xacro:joint name="${name}" id="${id}" bus="${bus}" kp="0.0" kd="1.0" second_encoder_source="-1" max_pos_limit="5000.0" min_pos_limit="-5000.0" actuator_trasmission="9"/>
+        <xacro:joint name="${name}" id="${id}" bus="${bus}" kp="0.0" kd="1.0" second_encoder_source="-1" max_pos_limit="5000.0" min_pos_limit="-5000.0" actuator_trasmission="9" max_current_A="40.0"/>
     </xacro:macro>
     <xacro:macro name="distributor_joint" params="name id">

File: src/pi3hat/pi3hat_hw_interface/urdf/omnicar_arm.xacro (robot description, xacro)
@@ -1,5 +1,5 @@
 <?xml version="1.0" ?>
 <robot name="omnicar"  xmlns:xacro="http://ros.org/wiki/xacro">
-    <xacro:macro name="joint" params="name id bus kp kd second_encoder_source max_pos_limit min_pos_limit actuator_trasmission">
+    <xacro:macro name="joint" params="name id bus kp kd second_encoder_source max_pos_limit min_pos_limit actuator_trasmission max_current_A">
         <joint name="${name}">
             <param name="id">${id}</param>
@@ -23,5 +23,5 @@
             <param name="second_encoder_trasmission">3.23076923</param>
             <param name="max_power_W">450</param>
-            <param name="max_current_A">40</param>
+            <param name="max_current_A">${max_current_A}</param>
             <param name="position_res">64</param>
             <param name="velocity_res">64</param>
@@ -42,8 +42,8 @@
     </xacro:macro>
     <xacro:macro name="arm_joint" params="name id bus">
-        <xacro:joint name="${name}" id="${id}" bus="${bus}" kp="100.0" kd="1.0" second_encoder_source="-1" max_pos_limit="3.14" min_pos_limit="-3.14" actuator_trasmission="9"/>
+        <xacro:joint name="${name}" id="${id}" bus="${bus}" kp="100.0" kd="1.0" second_encoder_source="-1" max_pos_limit="3.14" min_pos_limit="-3.14" actuator_trasmission="9" max_current_A="80.0"/>
     </xacro:macro>
     <xacro:macro name="wheel_joint" params="name id bus">
-        <xacro:joint name="${name}" id="${id}" bus="${bus}" kp="0.0" kd="1.0" second_encoder_source="-1" max_pos_limit="5000.0" min_pos_limit="-5000.0" actuator_trasmission="9"/>
+        <xacro:joint name="${name}" id="${id}" bus="${bus}" kp="0.0" kd="1.0" second_encoder_source="-1" max_pos_limit="5000.0" min_pos_limit="-5000.0" actuator_trasmission="9" max_current_A="40.0"/>
     </xacro:macro>
     <xacro:macro name="distributor_joint" params="name id">

File: src/pi3hat/pi3hat_hw_interface/urdf/omniquad12.xacro (robot description, xacro)
@@ -1,5 +1,5 @@
 <?xml version="1.0" ?>
 <robot name="omnicar"  xmlns:xacro="http://ros.org/wiki/xacro">
-    <xacro:macro name="joint" params="name id bus kp kd second_encoder_source max_pos_limit min_pos_limit actuator_trasmission">
+    <xacro:macro name="joint" params="name id bus kp kd second_encoder_source max_pos_limit min_pos_limit actuator_trasmission max_current_A">
         <joint name="${name}">
             <param name="id">${id}</param>
@@ -23,5 +23,5 @@
             <param name="second_encoder_trasmission">3.23076923</param>
             <param name="max_power_W">450</param>
-            <param name="max_current_A">40</param>
+            <param name="max_current_A">${max_current_A}</param>
             <param name="position_res">64</param>
             <param name="velocity_res">64</param>
@@ -41,9 +41,9 @@
         </joint>
     </xacro:macro>
-    <xacro:macro name="leg_joint" params="name id bus">
-        <xacro:joint name="${name}" id="${id}" bus="${bus}" kp="100.0" kd="1.0" second_encoder_source="-1" max_pos_limit="3.14" min_pos_limit="-3.14" actuator_trasmission="9"/>
+     <xacro:macro name="leg_joint" params="name id bus">
+        <xacro:joint name="${name}" id="${id}" bus="${bus}" kp="100.0" kd="1.0" second_encoder_source="-1" max_pos_limit="3.14" min_pos_limit="-3.14" actuator_trasmission="9" max_current_A="80.0"/>
     </xacro:macro>
     <xacro:macro name="wheel_joint" params="name id bus">
-        <xacro:joint name="${name}" id="${id}" bus="${bus}" kp="0.0" kd="1.0" second_encoder_source="-1" max_pos_limit="5000.0" min_pos_limit="-5000.0" actuator_trasmission="15"/>
+        <xacro:joint name="${name}" id="${id}" bus="${bus}" kp="0.0" kd="1.0" second_encoder_source="-1" max_pos_limit="5000.0" min_pos_limit="-5000.0" actuator_trasmission="15" max_current_A="40.0"/>
     </xacro:macro>
     <xacro:macro name="distributor_joint" params="name id">

Commit message: Update pi3hat hw interface and add Mazzolini arm
Squashed from branch 1-update-param:
- Update parameters (settable max voltage, flux brake margin)
- Update omniquad12_dji parameters
- Fix interface's problems to set params from xacro
- Add Mazzolini arm (urdf + controller config)
- Fix Mazzolini yaml
- Make max voltage and flux brake margin voltage settable, fix max power
- Update Log interface
- Tune omniquad12 actuator gains
- Tune activation hip angles and transition timing

Co-authored-by: Cionix90 <cionix90@gmail.com>
Co-authored-by: LoreMarti91 <martignettilorenzo@gmail.com>

File: src/pi3hat/pi3hat_hw_interface/urdf/SoftLeg.xacro (robot description, xacro)
@@ -1,5 +1,5 @@
 <?xml version="1.0" ?>
 <robot name="softleg" xmlns:xacro="http://ros.org/wiki/xacro">
-    <xacro:macro name="joint" params="name id bus kp kd second_encoder_source max_pos_limit min_pos_limit actuator_trasmission position_offset">
+    <xacro:macro name="joint" params="name id bus kp kd second_encoder_source max_pos_limit min_pos_limit actuator_trasmission position_offset max_current_A">
         <joint name="${name}">
             <param name="id">${id}</param>
@@ -22,4 +22,7 @@
             <param name="position_offset">${position_offset}</param>
             <param name="second_encoder_trasmission">3.23076923</param>
+            <param name="max_voltage">34.0</param>
+            <param name="flux_brake_margin_voltage">5.0</param>
+            <param name="max_current_A">${max_current_A}</param>
             <param name="position_res">64</param>
             <param name="velocity_res">64</param>
@@ -45,5 +48,5 @@
                      max_pos_limit="3.14" min_pos_limit="-3.14"
                      actuator_trasmission="9"
-                     position_offset="${position_offset}"/>
+                     position_offset="${position_offset}" max_current_A="80.0"/>
     </xacro:macro>
     <xacro:macro name="distributor_joint" params="name id">

File: src/pi3hat/pi3hat_hw_interface/urdf/arm.xacro (robot description, xacro)
@@ -1,5 +1,5 @@
 <?xml version="1.0" ?>
 <robot name="omnicar"  xmlns:xacro="http://ros.org/wiki/xacro">
-    <xacro:macro name="joint" params="name id bus kp kd second_encoder_source max_pos_limit min_pos_limit actuator_trasmission">
+    <xacro:macro name="joint" params="name id bus kp kd second_encoder_source max_pos_limit min_pos_limit actuator_trasmission max_current_A">
         <joint name="${name}">
             <param name="id">${id}</param>
@@ -22,4 +22,7 @@
             <param name="position_offset">0</param>
             <param name="second_encoder_trasmission">3.23076923</param>
+            <param name="max_voltage">34.0</param>
+            <param name="flux_brake_margin_voltage">5.0</param>
+            <param name="max_current_A">${max_current_A}</param>
             <param name="position_res">64</param>
             <param name="velocity_res">64</param>
@@ -40,8 +43,8 @@
     </xacro:macro>
     <xacro:macro name="arm_joint" params="name id bus">
-        <xacro:joint name="${name}" id="${id}" bus="${bus}" kp="100.0" kd="1.0" second_encoder_source="-1" max_pos_limit="3.14" min_pos_limit="-3.14" actuator_trasmission="9"/>
+        <xacro:joint name="${name}" id="${id}" bus="${bus}" kp="100.0" kd="1.0" second_encoder_source="-1" max_pos_limit="3.14" min_pos_limit="-3.14" actuator_trasmission="9" max_current_A="80.0"/>
     </xacro:macro>
     <xacro:macro name="wheel_joint" params="name id bus">
-        <xacro:joint name="${name}" id="${id}" bus="${bus}" kp="0.0" kd="1.0" second_encoder_source="-1" max_pos_limit="5000.0" min_pos_limit="-5000.0" actuator_trasmission="9"/>
+        <xacro:joint name="${name}" id="${id}" bus="${bus}" kp="0.0" kd="1.0" second_encoder_source="-1" max_pos_limit="5000.0" min_pos_limit="-5000.0" actuator_trasmission="9" max_current_A="40.0"/>
     </xacro:macro>
     <xacro:macro name="distributor_joint" params="name id">

File: src/pi3hat/pi3hat_hw_interface/urdf/arm_mazzolini.xacro (robot description, xacro)
@@ -1,4 +1,4 @@
 <?xml version="1.0" ?>
-<robot name="omnicar"  xmlns:xacro="http://ros.org/wiki/xacro">
+<robot name="mazzolini_arm"  xmlns:xacro="http://ros.org/wiki/xacro">
     <xacro:macro name="joint" params="name id bus kp kd second_encoder_source max_pos_limit min_pos_limit actuator_trasmission max_current_A">
         <joint name="${name}">
@@ -43,23 +43,5 @@
     </xacro:macro>
     <xacro:macro name="arm_joint" params="name id bus">
-        <xacro:joint name="${name}" id="${id}" bus="${bus}" kp="100.0" kd="1.0" second_encoder_source="-1" max_pos_limit="3.14" min_pos_limit="-3.14" actuator_trasmission="9" max_current_A="80.0"/>
-    </xacro:macro>
-    <xacro:macro name="wheel_joint" params="name id bus">
-        <xacro:joint name="${name}" id="${id}" bus="${bus}" kp="0.0" kd="1.0" second_encoder_source="-1" max_pos_limit="5000.0" min_pos_limit="-5000.0" actuator_trasmission="9" max_current_A="40.0"/>
-    </xacro:macro>
-    <xacro:macro name="distributor_joint" params="name id">
-        <joint name="${name}">
-            <param name="id">${id}</param>
-            <param name="bus">5</param>
-            <param name="type">power_dist</param>
-            <param name="voltage">64</param>
-            <param name="current">64</param>
-            <param name="temperature">64</param>
-            <param name="energy">0</param>
-            <param name="state">0</param>
-            <param name="switch_state">0</param>
-            <param name="lock_time">0</param>
-            <param name="boot_time">0</param>
-        </joint>
+        <xacro:joint name="${name}" id="${id}" bus="${bus}" kp="70.0" kd="1.0" second_encoder_source="-1" max_pos_limit="3.14" min_pos_limit="-3.14" actuator_trasmission="9" max_current_A="80.0"/>
     </xacro:macro>
     <ros2_control name="MoteusPi3Hat_Interface" type="system">
@@ -77,12 +59,6 @@
             <param name="attitude_hz">400</param>
         </hardware>
-        <xacro:wheel_joint name="LF_WHEEL" id="3" bus="2"/>
-        <xacro:wheel_joint name="RF_WHEEL" id="5" bus="4"/>
-        <xacro:wheel_joint name="LH_WHEEL" id="9" bus="1"/>
-        <xacro:wheel_joint name="RH_WHEEL" id="7" bus="3"/>
-        <xacro:arm_joint name="arm_pan" id="15" bus="4"/>
-        <xacro:arm_joint name="arm_tilt" id="16" bus="4"/>
-        <xacro:distributor_joint name="Distributor_L" id="32"/>
-        <xacro:distributor_joint name="Distributor_R" id="33"/>
+        <xacro:arm_joint name="joint1" id="3" bus="1"/>
+        <xacro:arm_joint name="joint2" id="4" bus="1"/>
     </ros2_control>
 </robot>

File: src/pi3hat/pi3hat_hw_interface/urdf/omnicar.xacro (robot description, xacro)
@@ -22,4 +22,7 @@
             <param name="position_offset">0.0</param>
             <param name="second_encoder_trasmission">3.23076923</param>
+            <param name="max_voltage">34.0</param>
+            <param name="flux_brake_margin_voltage">5.0</param>
+            <param name="max_current_A">40</param>
             <param name="position_res">64</param>
             <param name="velocity_res">64</param>

File: src/pi3hat/pi3hat_hw_interface/urdf/omniquad12.xacro (robot description, xacro)
@@ -1,5 +1,5 @@
 <?xml version="1.0" ?>
 <robot name="omnicar"  xmlns:xacro="http://ros.org/wiki/xacro">
-    <xacro:macro name="joint" params="name id bus kp kd second_encoder_source max_pos_limit min_pos_limit actuator_trasmission">
+    <xacro:macro name="joint" params="name id bus kp kd second_encoder_source max_pos_limit min_pos_limit actuator_trasmission max_current_A">
         <joint name="${name}">
             <param name="id">${id}</param>
@@ -22,4 +22,7 @@
             <param name="position_offset">0</param>
             <param name="second_encoder_trasmission">3.23076923</param>
+            <param name="max_voltage">34.0</param>
+            <param name="flux_brake_margin_voltage">5.0</param>
+            <param name="max_current_A">${max_current_A}</param>
             <param name="position_res">64</param>
             <param name="velocity_res">64</param>
@@ -39,9 +42,9 @@
         </joint>
     </xacro:macro>
-    <xacro:macro name="leg_joint" params="name id bus">
-        <xacro:joint name="${name}" id="${id}" bus="${bus}" kp="100.0" kd="1.0" second_encoder_source="-1" max_pos_limit="3.14" min_pos_limit="-3.14" actuator_trasmission="9"/>
+     <xacro:macro name="leg_joint" params="name id bus">
+     <xacro:joint name="${name}" id="${id}" bus="${bus}" kp="60.0" kd="0.6" second_encoder_source="-1" max_pos_limit="3.14" min_pos_limit="-3.14" actuator_trasmission="9" max_current_A="80.0"/>
     </xacro:macro>
     <xacro:macro name="wheel_joint" params="name id bus">
-        <xacro:joint name="${name}" id="${id}" bus="${bus}" kp="0.0" kd="1.0" second_encoder_source="-1" max_pos_limit="5000.0" min_pos_limit="-5000.0" actuator_trasmission="15"/>
+        <xacro:joint name="${name}" id="${id}" bus="${bus}" kp="0.0" kd="0.9" second_encoder_source="-1" max_pos_limit="5000.0" min_pos_limit="-5000.0" actuator_trasmission="15" max_current_A="40.0"/>
     </xacro:macro>
     <xacro:macro name="distributor_joint" params="name id">
